Commit message: 월드 추가

File: husky_customization/husky_custom_description/urdf/custom_description.urdf.xacro (robot description, xacro)
@@ -30,5 +30,5 @@
   <xacro:include filename="$(find velodyne_description)/urdf/HDL-32E.urdf.xacro"/>
   <xacro:HDL-32E parent="top_plate_link" name="velodyne" topic="/velodyne_points" hz="10" samples="2187" gpu="true">
-    <origin xyz="0.2 0 0.4" rpy="0 0 0" />
+    <origin xyz="0.2 0 1.0" rpy="0 0 0" />
   </xacro:HDL-32E>
 </robot>

Commit message: 월드 추가 및 laserscan 활용

File: husky_customization/husky_custom_description/urdf/custom_description.urdf.xacro (robot description, xacro)
@@ -30,5 +30,5 @@
   <xacro:include filename="$(find velodyne_description)/urdf/HDL-32E.urdf.xacro"/>
   <xacro:HDL-32E parent="top_plate_link" name="velodyne" topic="/velodyne_points" hz="10" samples="2187" gpu="true">
-    <origin xyz="0.2 0 1.0" rpy="0 0 0" />
+    <origin xyz="0.2 0 0.4" rpy="0 0 0" />
   </xacro:HDL-32E>
 </robot>
