Commit message: 미와성

File: husky_customization/husky_custom_description/urdf/custom_description_ouster_gps.urdf.xacro (robot description, xacro)
@@ -43,5 +43,6 @@
     <origin xyz="0 0 0.4" rpy="0 0 0"/>
   </xacro:OS1-32>
-  <!-- GPS 추가-->
+   <!-- GPS 추가-->
   <xacro:include filename="$(find husky_custom_description)/urdf/gps_sensor.urdf.xacro"/>
+  <xacro:gps_sensor parent="base_link"/>
 </robot>

File: husky_customization/husky_custom_description/urdf/gps_sensor.urdf.xacro (robot description, xacro)
@@ -1,57 +1,59 @@
-<!-- GPS 센서를 Husky에 추가하기 위한 URDF -->
 <?xml version="1.0"?>
 <robot xmlns:xacro="http://www.ros.org/wiki/xacro">
-  <!-- GPS 센서 링크 정의 -->
-  <link name="gps_link">
-    <visual>
-      <origin xyz="0 0 0" rpy="0 0 0"/>
-      <geometry>
-        <box size="0.05 0.05 0.02"/>
-      </geometry>
-      <material name="gps_material">
-        <color rgba="0.2 0.2 0.8 1.0"/>
-      </material>
-    </visual>
-    <collision>
-      <origin xyz="0 0 0" rpy="0 0 0"/>
-      <geometry>
-        <box size="0.05 0.05 0.02"/>
-      </geometry>
-    </collision>
-    <inertial>
-      <mass value="0.1"/>
-      <inertia ixx="0.001" ixy="0" ixz="0" iyy="0.001" iyz="0" izz="0.001"/>
-    </inertial>
-  </link>
-  <!-- GPS 센서를 base_link에 조인트로 연결 -->
-  <joint name="gps_joint" type="fixed">
-    <parent link="base_link"/>
-    <child link="gps_link"/>
-    <!-- Husky 뒤쪽 상단에 GPS 센서 위치 -->
-    <origin xyz="-0.3 0 0.3" rpy="0 0 0"/>
-  </joint>
-  <!-- Gazebo GPS 플러그인 -->
-  <gazebo reference="gps_link">
-    <sensor type="gps" name="husky_gps">
-      <pose>0 0 0 0 0 0</pose>
-      <visualize>true</visualize>
-      <update_rate>10.0</update_rate>
-      <plugin name="gps_controller" filename="libhector_gazebo_ros_gps.so">
-        <alwaysOn>true</alwaysOn>
-        <updateRate>10.0</updateRate>
-        <bodyName>gps_link</bodyName>
-        <frameId>gps_link</frameId>
-        <topicName>/gps/fix</topicName>
-        <velocityTopicName>/gps/fix_velocity</velocityTopicName>
-        <referenceLatitude>37.4419</referenceLatitude>
-        <referenceLongitude>-122.1430</referenceLongitude>
-        <referenceHeading>0</referenceHeading>
-        <referenceAltitude>10</referenceAltitude>
-        <drift>0.01 0.01 0.01</drift>
-        <gaussianNoise>0.1 0.1 0.1</gaussianNoise>
-        <velocityDrift>0 0 0</velocityDrift>
-        <velocityGaussianNoise>0.1 0.1 0.1</velocityGaussianNoise>
-      </plugin>
-    </sensor>
-  </gazebo>
+  <!-- GPS 매크로 정의 -->
+  <xacro:macro name="gps_sensor" params="parent">
+    <!-- GPS 센서 링크 정의 -->
+    <link name="gps_link">
+      <visual>
+        <origin xyz="0 0 0" rpy="0 0 0"/>
+        <geometry>
+          <box size="0.05 0.05 0.02"/>
+        </geometry>
+        <material name="gps_material">
+          <color rgba="0.2 0.2 0.8 1.0"/>
+        </material>
+      </visual>
+      <collision>
+        <origin xyz="0 0 0" rpy="0 0 0"/>
+        <geometry>
+          <box size="0.05 0.05 0.02"/>
+        </geometry>
+      </collision>
+      <inertial>
+        <mass value="0.1"/>
+        <inertia ixx="0.001" ixy="0" ixz="0" iyy="0.001" iyz="0" izz="0.001"/>
+      </inertial>
+    </link>
+    <!-- GPS 센서를 parent에 조인트로 연결 -->
+    <joint name="gps_joint" type="fixed">
+      <parent link="${parent}"/>
+      <child link="gps_link"/>
+      <!-- Husky 뒤쪽 상단에 GPS 센서 위치 -->
+      <origin xyz="-0.3 0 0.3" rpy="0 0 0"/>
+    </joint>
+    <!-- Gazebo GPS 플러그인 -->
+    <gazebo reference="gps_link">
+      <sensor type="gps" name="husky_gps">
+        <pose>0 0 0 0 0 0</pose>
+        <visualize>true</visualize>
+        <update_rate>10.0</update_rate>
+        <plugin name="gps_controller" filename="libhector_gazebo_ros_gps.so">
+          <alwaysOn>true</alwaysOn>
+          <updateRate>10.0</updateRate>
+          <bodyName>gps_link</bodyName>
+          <frameId>gps_link</frameId>
+          <topicName>/gps/fix</topicName>
+          <velocityTopicName>/gps/fix_velocity</velocityTopicName>
+          <referenceLatitude>37.4419</referenceLatitude>
+          <referenceLongitude>-122.1430</referenceLongitude>
+          <referenceHeading>0</referenceHeading>
+          <referenceAltitude>10</referenceAltitude>
+          <drift>0.01 0.01 0.01</drift>
+          <gaussianNoise>0.1 0.1 0.1</gaussianNoise>
+          <velocityDrift>0 0 0</velocityDrift>
+          <velocityGaussianNoise>0.1 0.1 0.1</velocityGaussianNoise>
+        </plugin>
+      </sensor>
+    </gazebo>
+  </xacro:macro>
 </robot>

Commit message: gps 추가중

File: husky_customization/husky_custom_description/urdf/custom_description_ouster_gps.urdf.xacro (robot description, xacro)
@@ -44,5 +44,7 @@
   </xacro:OS1-32>
    <!-- GPS 추가-->
+  <!-- GPS 센서 포함 -->
   <xacro:include filename="$(find husky_custom_description)/urdf/gps_sensor.urdf.xacro"/>
-  <xacro:gps_sensor parent="base_link"/>
+  <!-- Gazebo 플러그인 포함 -->
+  <xacro:include filename="$(find husky_custom_gazebo)/urdf/custom_description.gazebo.xacro"/>
 </robot>

File: husky_customization/husky_custom_description/urdf/gps_sensor.urdf.xacro (robot description, xacro)
@@ -1,35 +1,31 @@
 <?xml version="1.0"?>
 <robot xmlns:xacro="http://www.ros.org/wiki/xacro">
-  <!-- GPS 매크로 정의 -->
-  <xacro:macro name="gps_sensor" params="parent">
-    <!-- GPS 센서 링크 정의 -->
-    <link name="gps_link">
-      <visual>
-        <origin xyz="0 0 0" rpy="0 0 0"/>
-        <geometry>
-          <box size="0.05 0.05 0.02"/>
-        </geometry>
-        <material name="gps_material">
-          <color rgba="0.2 0.2 0.8 1.0"/>
-        </material>
-      </visual>
-      <collision>
-        <origin xyz="0 0 0" rpy="0 0 0"/>
-        <geometry>
-          <box size="0.05 0.05 0.02"/>
-        </geometry>
-      </collision>
-      <inertial>
-        <mass value="0.1"/>
-        <inertia ixx="0.001" ixy="0" ixz="0" iyy="0.001" iyz="0" izz="0.001"/>
-      </inertial>
-    </link>
-    <!-- GPS 센서를 parent에 조인트로 연결 -->
-    <joint name="gps_joint" type="fixed">
-      <parent link="${parent}"/>
-      <child link="gps_link"/>
-      <!-- Husky 뒤쪽 상단에 GPS 센서 위치 -->
-      <origin xyz="-0.3 0 0.3" rpy="0 0 0"/>
-    </joint>
-  </xacro:macro>
+  <!-- GPS Link -->
+  <link name="gps_link">
+    <inertial>
+      <mass value="0.001"/>
+      <origin xyz="0 0 0" rpy="0 0 0"/>
+      <inertia ixx="0.000000017" ixy="0" ixz="0"
+               iyy="0.000000017" iyz="0" izz="0.000000017"/>
+    </inertial>
+    <visual>
+      <origin xyz="0 0 0" rpy="0 0 0"/>
+      <geometry>
+        <box size="0.05 0.05 0.02"/>
+      </geometry>
+      <material name="black"/>
+    </visual>
+    <collision>
+      <origin xyz="0 0 0" rpy="0 0 0"/>
+      <geometry>
+        <box size="0.05 0.05 0.02"/>
+      </geometry>
+    </collision>
+  </link>
+  <!-- GPS Joint -->
+  <joint name="gps_joint" type="fixed">
+    <origin xyz="0.0 0.0 0.1" rpy="0 0 0"/>
+    <parent link="base_link"/>
+    <child link="gps_link"/>
+  </joint>
 </robot>

File: husky_customization/husky_custom_gazebo/urdf/custom_description.gazebo.xacro (robot description, xacro)
@@ -33,56 +33,19 @@
   <xacro:husky_robot_gazebo />
   <!-- GPS Gazebo 플러그인 추가 (월드 좌표 기준) -->
-    <gazebo reference="gps_link">
-      <sensor name="gps_sensor" type="gps">
-        <always_on>true</always_on>
-        <update_rate>10.0</update_rate>
-        <gps>
-          <position_sensing>
-            <horizontal>
-              <noise type="gaussian">
-                <mean>0.0</mean>
-                <stddev>2.0</stddev>
-              </noise>
-            </horizontal>
-            <vertical>
-              <noise type="gaussian">
-                <mean>0.0</mean>
-                <stddev>4.0</stddev>
-              </noise>
-            </vertical>
-          </position_sensing>
-          <velocity_sensing>
-            <horizontal>
-              <noise type="gaussian">
-                <mean>0.0</mean>
-                <stddev>0.1</stddev>
-              </noise>
-            </horizontal>
-            <vertical>
-              <noise type="gaussian">
-                <mean>0.0</mean>
-                <stddev>0.1</stddev>
-              </noise>
-            </vertical>
-          </velocity_sensing>
-        </gps>
-        <plugin name="gps_controller" filename="libhector_gazebo_ros_gps.so">
-          <alwaysOn>true</alwaysOn>
-          <updateRate>10.0</updateRate>
-          <bodyName>gps_link</bodyName>
-          <topicName>/ublox/fix</topicName>
-          <!-- 월드 파일의 좌표계에 맞춘 참조점 (위도 0, 경도 0) -->
-          <referenceLatitude>0.0</referenceLatitude>
-          <referenceLongitude>0.0</referenceLongitude>
-          <referenceHeading>0.0</referenceHeading>
-          <referenceAltitude>0.0</referenceAltitude>
-          <drift>0.001 0.001 0.001</drift>
-          <gaussianNoise>2.0 2.0 4.0</gaussianNoise>
-          <velocityDrift>0.001 0.001 0.001</velocityDrift>
-          <velocityGaussianNoise>0.1 0.1 0.1</velocityGaussianNoise>
-        </plugin>
-      </sensor>
-    </gazebo>
-  <xacro:include filename="$(find husky_custom_description)/urdf/custom_description_ouster_gps.urdf.xacro" />
+  <gazebo>
+    <plugin name="gps_controller" filename="libhector_gazebo_ros_gps.so">
+      <alwaysOn>true</alwaysOn>
+      <updateRate>10.0</updateRate>
+      <bodyName>base_link</bodyName>      <!-- gps_link 대신 base_link -->
+      <topicName>/ublox/fix</topicName>
+      <velocityTopicName>/ublox/fix_velocity</velocityTopicName>
+      <referenceLatitude>0.0</referenceLatitude>
+      <referenceLongitude>0.0</referenceLongitude>
+      <referenceHeading>0.0</referenceHeading>
+      <referenceAltitude>0.0</referenceAltitude>
+      <drift>0.0 0.0 0.0</drift>
+      <gaussianNoise>0.0 0.0 0.0</gaussianNoise>
+    </plugin>
+  </gazebo>
   <!-- Insert customizations below: -->
 </robot>
